Commit message: sticks

File: nao_description/urdf/nao_robot_v4_structure.urdf.xacro (robot description, xacro)
@@ -217,5 +217,10 @@
     <child link="CameraBottom_frame"/>
     <!-- rotated by 39.7 degrees -->
-    <origin xyz="0.05071 0 0.01774" rpy="-2.263692 0 -${pi_2}" />
+    <!--origin xyz="0.05071 0 0.01774" rpy="-2.263692 0 -${pi_2}" /-->
+    <!-- ramin & christian version -->
+    <!--
+    <origin xyz="0.05071 0 0.01774" rpy="-2.153692 0.02 -${pi_2-0.1}" />
+-->
+    <origin xyz="0.05071 0 0.01774" rpy="${-2.153692+0.04} 0.04 -${pi_2+0.00}" />
   </joint>
   <!-- Arm joints -->

Commit message: nao glockenspiel model

File: nao_description/urdf/nao_robot_v4_structure.urdf.xacro (robot description, xacro)
@@ -217,10 +217,6 @@
     <child link="CameraBottom_frame"/>
     <!-- rotated by 39.7 degrees -->
-    <!--origin xyz="0.05071 0 0.01774" rpy="-2.263692 0 -${pi_2}" /-->
-    <!-- ramin & christian version -->
-    <!--
+ <!--origin xyz="0.05071 0 0.01774" rpy="-2.263692 0 -${pi_2}" /-->
     <origin xyz="0.05071 0 0.01774" rpy="-2.153692 0.02 -${pi_2-0.1}" />
--->
-    <origin xyz="0.05071 0 0.01774" rpy="${-2.153692+0.04} 0.04 -${pi_2+0.00}" />
   </joint>
   <!-- Arm joints -->

Commit message: Parameterize the NaoV4 urdf.

File: nao_description/urdf/nao_robot_v4_structure.urdf.xacro (robot description, xacro)
@@ -191,5 +191,5 @@
     <child link="HeadYaw_link"/>
 	<!-- NeckOffsetZ -->
-    <origin xyz="0 0 0.1265" rpy="0 0 0" />
+    <origin xyz="0 0 0.1265" rpy="0 0 ${HeadYaw_y}" />
     <axis xyz="0 0 1" />
     <limit velocity="3.0" effort="30" lower="-2.0857" upper="2.0857" />
@@ -198,5 +198,5 @@
     <parent link="HeadYaw_link"/>
     <child link="HeadPitch_link"/>
-    <origin xyz="0 0 0" rpy="0 0 0" />
+    <origin xyz="0 0 0" rpy="0 ${HeadPitch_p} 0" />
     <axis xyz="0 1 0" />
     <limit velocity="3.0" effort="30" lower="-0.6720" upper="0.5149" />
@@ -217,13 +217,12 @@
     <child link="CameraBottom_frame"/>
     <!-- rotated by 39.7 degrees -->
- <!--origin xyz="0.05071 0 0.01774" rpy="-2.263692 0 -${pi_2}" /-->
-    <origin xyz="0.05071 0 0.01774" rpy="-2.153692 0.02 -${pi_2-0.1}" />
+    <origin xyz="${Camera_tx} ${Camera_ty} ${Camera_tz}" rpy="${Camera_rr} ${Camera_rp} ${Camera_ry}" />
   </joint>
   <!-- Arm joints -->
-  <xacro:macro name="arm_joints" params="side reflect">
+  <xacro:macro name="arm_joints" params="side reflect ShoulderPitch_p ElbowYaw_r">
   <joint name="${side}ShoulderPitch" type="revolute">
     <parent link="torso"/>
     <child link="${side}ShoulderPitch_link"/>
-    <origin xyz="0 ${reflect*-0.098} 0.1" rpy="0 0 0"/>
+    <origin xyz="0 ${reflect*-0.098} 0.1" rpy="0 ${ShoulderPitch_p} 0"/>
     <axis xyz="0 1 0"/>
     <limit velocity="3.0" effort="30" lower="-2.0857" upper="2.0857"/>

Commit message: parameterized nao_robot_v4_structure.urdf.xacro

File: nao_description/urdf/nao_robot_v4_structure.urdf.xacro (robot description, xacro)
@@ -231,5 +231,5 @@
     <parent link="${side}ShoulderRoll_link"/>
     <child link="${side}ElbowYaw_link"/>
-    <origin xyz="0.105 ${reflect*-0.015} 0" rpy="0 0 0"/>
+    <origin xyz="0.105 ${reflect*-0.015} 0" rpy="${ElbowYaw_r} 0 0"/>
     <axis xyz="1 0 0"/>
     <limit velocity="3.0" effort="30" lower="-2.0857" upper="2.0857"/>
@@ -246,10 +246,10 @@
     <parent link="LWristYaw_link" />
     <child link="l_wrist" />
-    <origin xyz="0 0 0" />
+    <origin xyz="0 0 0" rpy="0 0 0" />
   </joint>
   <joint name="r_wrist_joint" type="fixed">
     <parent link="RWristYaw_link" />
     <child link="r_wrist" />
-    <origin xyz="0 0 0" />
+    <origin xyz="0 0 0" rpy="0 0 0"/>
   </joint>
   <joint name="l_gripper_joint" type="fixed">
@@ -266,5 +266,5 @@
     <parent link="LElbowYaw_link"/>
     <child link="LElbowRoll_link"/>
-    <origin xyz="0 0 0" rpy="0 0 0"/>
+    <origin xyz="0 0 0" rpy="0 0 ${LElbowRoll_y}"/>
     <axis xyz="0 0 1"/>
     <limit velocity="3.0" effort="30" lower="-1.5446" upper="-0.0349"/>
@@ -273,5 +273,5 @@
     <parent link="RElbowYaw_link"/>
     <child link="RElbowRoll_link"/>
-    <origin xyz="0 0 0" rpy="0 0 0"/>
+    <origin xyz="0 0 0" rpy="0 0 ${RElbowRoll_y}"/>
     <axis xyz="0 0 1"/>
     <limit velocity="3.0" effort="30" lower="0.0349" upper="1.5446"/>
@@ -280,5 +280,5 @@
     <parent link="LShoulderPitch_link"/>
     <child link="LShoulderRoll_link"/>
-    <origin xyz="0 0 0" rpy="0 0 0"/>
+    <origin xyz="0 0 0" rpy="0 0 ${LShoulderRoll_y}"/>
     <axis xyz="0 0 1"/>
     <limit velocity="3.0" effort="30" lower="-0.3142" upper="1.3265"/>
@@ -287,10 +287,10 @@
     <parent link="RShoulderPitch_link"/>
     <child link="RShoulderRoll_link"/>
-    <origin xyz="0 0 0" rpy="0 0 0"/>
+    <origin xyz="0 0 0" rpy="0 0 ${RShoulderRoll_y}"/>
     <axis xyz="0 0 1"/>
     <limit velocity="3.0" effort="30" lower="-1.3265" upper="0.3142"/>
   </joint>
-  <xacro:arm_joints side="L" reflect="-1"/>
-  <xacro:arm_joints side="R" reflect="1"/>
+  <xacro:arm_joints side="L" reflect="-1" ShoulderPitch_p="${LShoulderPitch_p}" ElbowYaw_r="${LElbowYaw_r}" />
+  <xacro:arm_joints side="R" reflect="1" ShoulderPitch_p="${RShoulderPitch_p}" ElbowYaw_r="${RElbowYaw_r}" />
   <!-- Leg joints -->
   <joint name="LHipYawPitch" type="revolute">
